File: AxxSolder.kicad_pcb (KiCad board)
At the start: 2 copper layers, 39 x 71 mm, 111 parts, among them IC1 LTC4440AHMS8E-5#PBF, IC2 STM32G431KBT6, IC4 OPA2333AIDRBR, IC5 STM32G431KBT6, IC6 TPS54302DDCR, IC7 STUSB4500QTR, IC8 USBLC6-2P6, J1 Conn_01x07_Male, J2 USB_B_Micro, J5 USB4105-GF-A-120, J6 Conn_01x06_Socket, Q1 STL9P3LLH6, Q2 2N7002NXAKR, U1 PEC11L-4220F-S0015, U2 BSC014N04LS

Commit message: update filestructure for AxxSolder V3.0 and forward
Parts:
- removed J2: USB_B_Micro, USB3140-30-0230-1-C_REVE1:GCT_USB3140-30-0230-1-C_REVE1
- added C32: 10u, Capacitor_SMD:C_0805_2012Metric, F.Cu at (90.1, 70.6)
- added C33: 1u, Capacitor_SMD:C_0805_2012Metric, F.Cu at (87.7, 98.0)
- added C34: 100n, Capacitor_SMD:C_0805_2012Metric, F.Cu at (87.7, 101.0)
- added C35: 100n, Capacitor_SMD:C_0805_2012Metric, F.Cu at (64.8, 98.5)
- added C36: 100n, Capacitor_SMD:C_0805_2012Metric, F.Cu at (64.8, 101.5)
- added C37: 100n, Capacitor_SMD:C_0805_2012Metric, F.Cu at (64.8, 104.5)
- added D11: BAV199WQ-7, Library:SOT65P210X110-3N, F.Cu at (86.8, 83.6)
- added D4: SMBJ24A, footprints:DIOM5436X261N, F.Cu at (84.0, 105.6)
- added D5: BAV199WQ-7, Library:SOT65P210X110-3N, F.Cu at (86.8, 79.8)
- added D6: ESDA25W, footprints:SOT65P210X110-3N, F.Cu at (87.2, 110.2)
- added D8: ESDA25P35, footprints:ESDA25P351U1M, F.Cu at (82.3, 110.4)
- added FB1: BLM18HE601SN1D, footprints:BLM18SP221SN1B, F.Cu at (89.9, 73.3)
- added FB1: BLM18HE601SN1D, footprints:BLM18SP221SN1B, F.Cu at (91.2, 79.2)
- added IC3: OPA2387DSGT, footprints:SON50P200X200X80-9N, F.Cu at (64.7, 108.2)
- added J4: 691243110008, footprints:691243110008, F.Cu at (72.4, 66.2)
- added Q2: 2N7002NXAKR, Library:SOT95P230X110-3N, F.Cu at (69.4, 103.8)
- added Q5: STL9P3LLH6, footprints:STL20N6F7, F.Cu at (82.7, 99.5)
- added R21: 10k, Resistor_SMD:R_0805_2012Metric, F.Cu at (60.3, 98.5)
- added R34: 10k, Resistor_SMD:R_0805_2012Metric, F.Cu at (77.7, 98.0)
- added R36: 1k, Resistor_SMD:R_0805_2012Metric, F.Cu at (77.7, 101.0)
- added R37: 4k7, Resistor_SMD:R_0805_2012Metric, F.Cu at (77.7, 103.9)
- added R38: 22k, Resistor_SMD:R_0805_2012Metric, F.Cu at (77.7, 106.9)
- added R39: 360k, Resistor_SMD:R_0805_2012Metric, F.Cu at (60.3, 101.4)
- added R40: 10k, Resistor_SMD:R_0805_2012Metric, F.Cu at (60.3, 104.4)
- added R41: 10k, Resistor_SMD:R_0805_2012Metric, F.Cu at (60.3, 107.3)
- added U3: TPD2E2U06QDBZRQ1, footprints:SOT95P237X95-3N, F.Cu at (69.5, 99.3)
- added U3: OPA2376xxYZD, Package_BGA:Texas_DSBGA-8_0.9x1.9mm_Layout2x4_P0.5mm, F.Cu at (91.7, 113.7)
- C5: value 10u -> 4.7u
- IC1: value LTC4440AHMS8E-5#PBF -> LTC4440AHMS8E; footprint LTC4440AHMS8E-5#PBF:SOP65P490X110-9N -> footprints:SOP65P490X110-9N
- IC4: value OPA2333AIDRBR -> OPA2387DSGT; footprint OPA2333AIDRBR:SON65P300X300X100-9N-D -> footprints:SON65P300X300X100-9N-D; moved to F.Cu
- IC7: footprint STUSB4500QTR:QFN50P400X400X100-25N-D -> footprints:QFN50P400X400X100-25N-D
- L1: value SRP7028CC-100M -> SRP7028CC
- R21, R22: value 470k -> 360k
- R33: value 100k -> 100
- TP5: value Thermocouple_TP -> TC_TP
- moved IC4 32.9 mm to (82.0, 73.6)
Connections:
- net /Busvoltage renamed /VDD_inp
- net /Current_2 renamed /SW_3
- net /Heater_1 renamed /Heater
- net /Identification_inp renamed /SD_CS
- C11 pad 1: +3.3V -> Net-(IC2-VDDA)
- C12 pad 1: +3.3V -> Net-(IC2-VDDA)
- C15 pad 1: /Thermocouple_1 -> /TC
- C16 pad 1: /Current_1 -> /Current
- C20 pad 1: Net-(IC7-VREG_2V7) -> /VBUS
- C28 pad 1: /Handle_inp -> /Handle_sense2
- C29 pad 1: /Stand_inp -> /Stand_sense
- C30 pad 1: Net-(IC7-VREG_1V2) -> Net-(IC7-VREG_2V7)
- C31 pad 2: VDD -> /VDD_IN
- C8 pad 1: /ENC_Button -> /SW1
- D3 pad 3: /Handle_inp -> /Handle_inp2
- D4 pad 6: GND -> /SPI_CS
- IC2 pad 10: /Thermocouple_2 -> /SW1
- IC2 pad 15: +3.3V -> Net-(IC2-VDDA)
- IC2 pad 18: /HEATER_2 -> /Handle_inp2
- IC2 pad 19: /Handle_inp -> /Handle_inp1
- IC2 pad 29: /ENC_Button -> /SPI_CS
- IC2 pad 5: /Thermocouple_1 -> /TC
- IC2 pad 6: /Current_1 -> /Current
- IC2 pad 7: /MCU_TX -> /SW_2
- IC4 pad 2: Net-(D5-common) -> Net-(IC4--IN_A)
- IC4 pad 3: Net-(D6-common) -> Net-(IC4-+IN_A)
- IC5 pad 10: /Thermocouple_2 -> /SW1
- IC5 pad 15: +3.3V -> Net-(IC2-VDDA)
- IC5 pad 18: /HEATER_2 -> /Handle_inp2
- IC5 pad 19: /Handle_inp -> /Handle_inp1
- IC5 pad 29: /ENC_Button -> /SPI_CS
- IC5 pad 5: /Thermocouple_1 -> /TC
- IC5 pad 6: /Current_1 -> /Current
- IC5 pad 7: /MCU_TX -> /SW_2
- IC7 pad 1: Net-(D10-CATHODE_2) -> /CC1
- IC7 pad 11: unconnected-(IC7-ATTACH-Pad11) -> (no net)
- IC7 pad 14: unconnected-(IC7-POWER_OK3-Pad14) -> (no net)
- IC7 pad 15: unconnected-(IC7-GPIO-Pad15) -> (no net)
- IC7 pad 17: unconnected-(IC7-A_B_SIDE-Pad17) -> (no net)
- IC7 pad 19: unconnected-(IC7-ALERT-Pad19) -> (no net)
- IC7 pad 2: Net-(D10-CATHODE_2) -> /CC1
- IC7 pad 20: unconnected-(IC7-POWER_OK2-Pad20) -> (no net)
- IC7 pad 3: unconnected-(IC7-NC-Pad3) -> (no net)
- IC7 pad 4: Net-(D10-CATHODE_1) -> /CC2
- IC7 pad 5: Net-(D10-CATHODE_1) -> /CC2
- IC8 pad 5: /V_BUS -> +5V
- J5 pad A6: Net-(J5-DP1) -> /USB_DP
- J5 pad A7: Net-(J5-DN1) -> /USB_DN
- J5 pad B6: Net-(J5-DP1) -> /USB_DP
- J5 pad B7: Net-(J5-DN1) -> /USB_DN
- Q1 pad 5: Net-(D13-A) -> /VDD_IN
- R12 pad 2: /ENC_Button -> /SW1
- R15 pad 2: Net-(Q2-Pad1) -> Net-(Q2-G)
- R16 pad 1: Net-(Q2-Pad1) -> Net-(Q2-G)
- R19 pad 2: Net-(D5-common) -> Net-(IC3A--)
- R20 pad 2: Net-(D6-common) -> Net-(IC3A-+)
- R21 pad 1: Net-(D6-common) -> Net-(IC4-+IN_A)
- R22 pad 1: /Thermocouple_1 -> /TC
- R22 pad 2: Net-(D5-common) -> Net-(IC3A--)
- R23 pad 1: Net-(IC4-+IN_B) -> Net-(IC3B-+)
- R24 pad 1: Net-(IC4--IN_B) -> /Current
- R24 pad 2: /Current_1 -> Net-(IC3B--)
- R25 pad 1: Net-(IC4-+IN_B) -> /BLUE
- R25 pad 2: /BLUE -> Net-(IC3B-+)
- R26 pad 1: GND -> Net-(IC3B--)
- R26 pad 2: Net-(IC4--IN_B) -> GND
- R27 pad 1: /SCL -> /SDA
- R30 pad 1: /SDA -> /SCL
- R32 pad 2: /USB_PD_GATE -> Net-(Q5-G)
- R33 pad 1: /USB_PD_GATE -> Net-(Q5-G)
- R33 pad 2: /VBUS -> Net-(C31-Pad1)
- R35 pad 1: Net-(IC7-DISCH) -> /VDD_IN
- R35 pad 2: VDD -> Net-(IC7-DISCH)
- R6 pad 1: /Handle_inp -> /Handle_inp2
- R6 pad 2: /Handle_sense -> /Handle_sense2
- R9 pad 2: /Handle_sense -> /Handle_sense2
- TP5 pad 1: /Thermocouple_1 -> /TC
- TP6 pad 1: /Current_1 -> /Current
- U1 pad 1: /ENC_Button -> /SW1
Routing:
- net /SPI_CS: track 0.00 -> 65.5 mm, vias 0 -> 4
- net /ENC_Button: track 65.5 -> 0.00 mm, vias 4 -> 0
- net /Handle_inp: track 28.3 -> 0.00 mm, vias 1 -> 0
- net (no net): track 0.00 -> 28.3 mm
- net Net-(IC4--IN_B): track 6.40 -> 0.00 mm
- net GND: track 508.9 -> 515.3 mm
- net Net-(IC4-+IN_B): track 4.23 -> 0.00 mm
- net /BLUE: track 29.8 -> 34.0 mm
- net /Thermocouple_2: track 2.39 -> 0.00 mm
- net /SW1: track 0.00 -> 2.39 mm
- net /Handle_inp2: track 0.00 -> 2.31 mm, vias 0 -> 1
- net /HEATER_2: track 2.31 -> 0.00 mm
- net Net-(D6-common): track 14.7 -> 12.8 mm
- net Net-(J5-DP1): vias 2 -> 0
- net Net-(J5-DN1): vias 2 -> 0
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