File: AxxSolder.kicad_pcb (KiCad board)
At the start: 2 copper layers, 39 x 71 mm, 137 parts, among them IC1 LTC4440AHMS8E, IC2 STM32G431KBT6, IC3 OPA2387DSGT, IC4 OPA2387DSGT, IC5 STM32G431KBT6, IC6 TPS54302DDCR, IC7 STUSB4500QTR, IC8 USBLC6-2P6, J1 Conn_01x07_Male, J4 691243110008, J5 USB4105-GF-A-120, J6 Conn_01x06_Socket, Q1 STL9P3LLH6, Q2 2N7002NXAKR, Q5 STL9P3LLH6, U1 PEC11L-4220F-S0015, U2 BSC014N04LS, U3 OPA2376xxYZD, U3 TPD2E2U06QDBZRQ1

Commit message: multiple updates for AxxSolder hw 3.0
Parts:
- removed C23: 330u, EMZR500ARA331MJA0G:CAPAE1030X1050N
- removed the C30 at (118.0, 109.3)
- removed the C31 at (128.3, 115.8)
- removed the C35 at (64.8, 98.5)
- removed the C36 at (64.8, 101.5)
- removed the C37 at (64.8, 104.5)
- removed the D11 at (86.8, 83.6)
- removed the D11 at (132.3, 88.8)
- removed D13: V7NM103-M3_I, V7NM103-M3_I:V7NM103M3I
- removed the D4 at (84.0, 105.6)
- removed the D4 at (116.5, 56.3)
- removed the D5 at (86.8, 79.8)
- removed the D5 at (110.9, 74.0)
- removed the D6 at (87.2, 110.2)
- removed the D8 at (82.3, 110.4)
- removed the D8 at (112.7, 109.5)
- removed F2: 0154007.DRL, 0154007:0154100DR
- removed the FB1 at (89.9, 73.3)
- removed the FB1 at (91.2, 79.2)
- removed H3, H4: MountingHole, MountingHole:MountingHole_3mm
- removed the IC5 at (125.5, 69.8)
- removed IC7: STUSB4500QTR, footprints:QFN50P400X400X100-25N-D
- removed IC8: USBLC6-2P6, USBLC6-2P6:USBLC62P6
- removed J5: USB4105-GF-A-120, USB4105-GF-A:GCT_USB4105-GF-A-120
- removed J6: Conn_01x06_Socket, Connector_PinSocket_2.54mm:PinSocket_1x06_P2.54mm_Vertical
- removed JP1, JP2: SolderJumper_2_Open, Jumper:SolderJumper-2_P1.3mm_Open_TrianglePad1.0x1.5mm
- removed the Q2 at (121.8, 104.5)
- removed the Q2 at (69.4, 103.8)
- removed Q5: STL9P3LLH6, footprints:STL20N6F7
- removed the R16 at (121.5, 101.5)
- removed the R17 at (121.5, 107.5)
- removed the R21 at (60.3, 98.5)
- removed the R21 at (108.2, 77.5)
- removed the R22 at (108.2, 73.9)
- removed the R26 at (120.8, 78.2)
- removed the R31 at (122.9, 113.6)
- removed the R34 at (125.6, 116.6)
- removed the R34 at (77.7, 98.0)
- removed the R35 at (123.5, 113.5)
- removed R36: 1k, Resistor_SMD:R_0805_2012Metric
- removed R37: 4k7, Resistor_SMD:R_0805_2012Metric
- removed R38: 22k, Resistor_SMD:R_0805_2012Metric
- removed R41: 10k, Resistor_SMD:R_0805_2012Metric
- removed TP3: GND_TP, TestPoint:TestPoint_THTPad_D1.0mm_Drill0.5mm
- removed the TP5 at (124.7, 77.7) (x2)
- removed the TP6 at (122.7, 76.5) (x2)
- removed U2: BSC014N04LS, BSC014N04LS:BSC014N04LS
- removed the U3 at (69.5, 99.3)
- removed the U3 at (91.7, 113.7)
- added C1: 100n, Capacitor_SMD:C_0603_1608Metric, B.Cu at (166.5, 88.2)
- added C17: 1u, Capacitor_SMD:C_0603_1608Metric, B.Cu at (189.7, 137.2)
- added C18: 1u, Capacitor_SMD:C_0603_1608Metric, B.Cu at (189.7, 135.8)
- added C19: 10u, Capacitor_SMD:C_0603_1608Metric, B.Cu at (191.8, 143.5)
- added C28: 100n, Capacitor_SMD:C_0603_1608Metric, F.Cu at (190.2, 135.2)
- added C29: 100n, Capacitor_SMD:C_0603_1608Metric, B.Cu at (166.9, 97.0)
- added C4: 100n, Capacitor_SMD:C_0603_1608Metric, B.Cu at (164.8, 76.0)
- added D1: BAV199WQ-7, footprints:SOT65P210X110-3N, B.Cu at (186.5, 93.7)
- added D11: ESDA25P35, footprints:ESDA25P351U1M, B.Cu at (191.2, 141.2)
- added D3: ESDA25W, footprints:SOT65P210X110-3N, B.Cu at (189.0, 143.5)
- added D4: SMBJ24A, footprints:DIOM5436X261N, B.Cu at (177.5, 71.0)
- added F1: 0154007.DRL, footprints:0154100DR, B.Cu at (187.2, 71.0)
- added FB1: BLM18HE601SN1D, Resistor_SMD:R_0603_1608Metric, B.Cu at (182.7, 106.4)
- added G***: LOGO, LOGO, F.Cu at (180.5, 85.0)
- added IC1: OPA2387DSGT, footprints:SON50P200X200X80-9N, B.Cu at (182.5, 100.5)
- added J2: 691243110009, footprints:691243110009, B.Cu at (196.2, 106.0)
- added J3: Conn_01x05_Socket, Connector_PinSocket_2.54mm:PinSocket_1x05_P2.54mm_Vertical, B.Cu at (162.5, 113.9)
- added Q2: 2N7002NXAKR, footprints:SOT95P230X110-3N, B.Cu at (163.0, 139.8)
- added Q3: STL10N3LLH5, footprints:STL10N3LLH5, B.Cu at (197.7, 130.4)
- added R15: 1k, Resistor_SMD:R_0603_1608Metric, B.Cu at (185.2, 133.8)
- added R18: 4k7, Resistor_SMD:R_0603_1608Metric, B.Cu at (195.2, 111.2)
- added R21: 47k, Resistor_SMD:R_0603_1608Metric, B.Cu at (166.9, 95.5)
- added R34: 4k7, Resistor_SMD:R_0603_1608Metric, B.Cu at (168.5, 139.8)
- added R4: 4k7, Resistor_SMD:R_0603_1608Metric, B.Cu at (183.5, 93.8)
- added R5: 1k5, Resistor_SMD:R_0603_1608Metric, B.Cu at (189.0, 96.6)
- added R6: 100k, Resistor_SMD:R_0603_1608Metric, B.Cu at (169.2, 71.0)
- added R7: 4k7, Resistor_SMD:R_0603_1608Metric, B.Cu at (182.0, 93.8)
- added R8: 360k, Resistor_SMD:R_0603_1608Metric, B.Cu at (182.7, 98.2)
- added R9: 220k, Resistor_SMD:R_0603_1608Metric, B.Cu at (182.8, 96.0)
- added REF**: PinHeader_1x02_P2.54mm_Vertical, Connector_PinHeader_2.54mm:PinHeader_1x02_P2.54mm_Vertical, F.Cu at (162.2, 72.2)
- added REF**: PinHeader_1x02_P2.54mm_Vertical, Connector_PinHeader_2.54mm:PinHeader_1x02_P2.54mm_Vertical, F.Cu at (198.8, 72.2)
- added S1: ADTSM644KVTR, footprints:ADTSM644KVTR, F.Cu at (170.2, 135.4)
- added S3: ADTSM644KVTR, footprints:ADTSM644KVTR, F.Cu at (196.2, 135.4)
- added TP1: VDD_TP, TestPoint:TestPoint_THTPad_D1.0mm_Drill0.5mm, B.Cu at (163.5, 88.8)
- added TP10: DIAG_TP, TestPoint:TestPoint_Pad_D1.0mm, B.Cu at (188.2, 113.2)
- added TP11: DIAG_TP, TestPoint:TestPoint_Pad_D1.0mm, B.Cu at (187.2, 127.5)
- added TP12: DIAG_TP, TestPoint:TestPoint_Pad_D1.0mm, B.Cu at (195.2, 127.5)
- added TP2: 3.3V_TP, TestPoint:TestPoint_THTPad_D1.0mm_Drill0.5mm, B.Cu at (166.8, 91.2)
- added TP4: Current_TP, TestPoint:TestPoint_Pad_D1.0mm, B.Cu at (179.5, 102.8)
- added TP5: TC_TP, TestPoint:TestPoint_Pad_D1.0mm, B.Cu at (187.5, 106.2)
- added TP6: GND_TP, TestPoint:TestPoint_THTPad_D1.0mm_Drill0.5mm, B.Cu at (173.5, 68.8)
- added U3: PEC11J-9220F-S0015, footprints:PEC11J9220FS0015, F.Cu at (170.2, 135.4)
- added U4: BSC014N04LS, footprints:BSC014N04LS, B.Cu at (186.5, 76.3)
- added Y1: NX2016SA-32M-EXS00A-CS06465, footprints:NX2016SA32MEXS00ACS06465, B.Cu at (178.4, 109.2)
- C10: value 100n -> 1n; footprint Capacitor_SMD:C_0805_2012Metric -> Capacitor_SMD:C_0603_1608Metric; moved to B.Cu
- C11: value 100n -> 1n; footprint Capacitor_SMD:C_0805_2012Metric -> Capacitor_SMD:C_0603_1608Metric
- C12: value 10u -> 10p; footprint Capacitor_SMD:C_0805_2012Metric -> Capacitor_SMD:C_0603_1608Metric
- C13, C22, C6: footprint Capacitor_SMD:C_0805_2012Metric -> Capacitor_SMD:C_0603_1608Metric; moved to B.Cu
- C14: value 10u -> 100n; footprint Capacitor_SMD:C_0805_2012Metric -> Capacitor_SMD:C_0603_1608Metric
- C15: value 1n -> 10u; footprint Capacitor_SMD:C_0805_2012Metric -> Capacitor_SMD:C_0603_1608Metric
- C16: value 1n -> 1u; footprint Capacitor_SMD:C_0805_2012Metric -> Capacitor_SMD:C_0603_1608Metric
- C2: renamed from C19; footprint Capacitor_SMD:C_0805_2012Metric -> Capacitor_SMD:C_0603_1608Metric; moved to B.Cu
- C20: value 1u -> 100n; footprint Capacitor_SMD:C_0805_2012Metric -> Capacitor_SMD:C_0603_1608Metric; moved to B.Cu
- C21, C24, C34: footprint Capacitor_SMD:C_0805_2012Metric -> Capacitor_SMD:C_0603_1608Metric
- C25: value 22u -> 10u; footprint Capacitor_SMD:C_1206_3216Metric -> Capacitor_SMD:C_0603_1608Metric
- C26: value 75p -> 100n; footprint Capacitor_SMD:C_0805_2012Metric -> Capacitor_SMD:C_0603_1608Metric; moved to F.Cu
- C27: value 22u -> 100n; footprint Capacitor_SMD:C_1206_3216Metric -> Capacitor_SMD:C_0603_1608Metric; moved to F.Cu
- C3: value 100n -> 10p; footprint Capacitor_SMD:C_0805_2012Metric -> Capacitor_SMD:C_0603_1608Metric
- C30: renamed from C29; footprint Capacitor_SMD:C_0805_2012Metric -> Capacitor_SMD:C_0603_1608Metric; moved to B.Cu
- C31: renamed from C28; footprint Capacitor_SMD:C_0805_2012Metric -> Capacitor_SMD:C_0603_1608Metric; moved to B.Cu
- C32: value 10u -> 100n; footprint Capacitor_SMD:C_0805_2012Metric -> Capacitor_SMD:C_0603_1608Metric; moved to B.Cu
- C33: value 1u -> 100n; footprint Capacitor_SMD:C_0805_2012Metric -> Capacitor_SMD:C_0603_1608Metric
- C36: renamed from C1; footprint Capacitor_SMD:C_0805_2012Metric -> Capacitor_SMD:C_0603_1608Metric
- C37: renamed from C2; footprint Capacitor_SMD:C_0805_2012Metric -> Capacitor_SMD:C_0603_1608Metric
- C5: value 4.7u -> 100n; footprint Capacitor_SMD:C_0805_2012Metric -> Capacitor_SMD:C_0603_1608Metric
- C7: value 100n -> 75p; footprint Capacitor_SMD:C_0805_2012Metric -> Capacitor_SMD:C_0603_1608Metric
- C8, C9: value 100n -> 22u; footprint Capacitor_SMD:C_0805_2012Metric -> Capacitor_SMD:C_1206_3216Metric; moved to B.Cu
- D10: value ESDA25W -> PMEG10030ELPX; footprint ESDA25W:SOT65P210X110-3N -> footprints:SODFL4725X110N
- D12: value BAT54S -> TPD2E2U06; footprint BAT54S,215:SOT95P230X110-3N -> footprints:SOT95P237X95-3N
- D2: value PMEG6020ER -> BAV199WQ-7; footprint PMEG6020ER,115:PMEG6020ER115 -> footprints:SOT65P210X110-3N
- D5: renamed from D6; footprint BAT54S,215:SOT95P230X110-3N -> footprints:SOT95P230X110-3N
- D6: renamed from D3; footprint BAT54S,215:SOT95P230X110-3N -> footprints:SOT95P230X110-3N
- D7: value PMEG10030ELPX -> BAT54S; footprint PMEG10030ELPX:SODFL4725X110N -> footprints:SOT95P230X110-3N; moved to B.Cu
- D8: renamed from D1; footprint BAT54S,215:SOT95P230X110-3N -> footprints:SOT95P230X110-3N
- D9: value SMBJ24CA -> PMEG6020ER; footprint SMBJ24CA:DIOM5436X261N -> footprints:PMEG6020ER115; moved to B.Cu
- H1: footprint MountingHole:MountingHole_3mm -> MountingHole:MountingHole_2.5mm; moved to F.Cu
- H2: footprint MountingHole:MountingHole_3mm -> MountingHole:MountingHole_2.5mm
- IC2: value STM32G431KBT6 -> STM32F303CCT6TR; footprint STM32G431KBT6:QFP80P900X900X160-32N -> footprints:QFP50P900X900X160-48N
- IC3: value OPA2387DSGT -> TPS54302DDCR; footprint footprints:SON50P200X200X80-9N -> footprints:SOT95P280X110-6N; moved to B.Cu
- IC4: value OPA2387DSGT -> STUSB4500QTR; footprint footprints:SON65P300X300X100-9N-D -> footprints:QFN50P400X400X100-25N-D; moved to B.Cu
- IC6: value TPS54302DDCR -> MAX16171ATA_VY+T; footprint TPS54302DDCR:SOT95P280X110-6N -> footprints:SON50P300X200X80-9N
- J1: value Conn_01x07_Male -> USB4110-GF-A; footprint 691243310007:691243310007 -> footprints:USB4110GFA
- J4: value 691243110008 -> Conn_01x02_Pin; footprint footprints:691243110008 -> Connector_PinHeader_1.27mm:PinHeader_1x02_P1.27mm_Vertical; moved to B.Cu
- L1: footprint SRP7028CC-100M:INDPM7366X300N -> footprints:INDPM7366X300N
- LS1: footprint CMI-9653S-SMT-TR:CMI9653SSMTTR -> footprints:CMI9653SSMTTR; moved to B.Cu
- PS1: footprint LD1117AS33TR:SOT230P700X190-4N -> footprints:SOT230P700X190-4N; moved to B.Cu
- Q1: footprint STL9P3LLH6:STL20N6F7 -> footprints:STL20N6F7
- R1: value 4k7 -> 1k5; footprint Resistor_SMD:R_0805_2012Metric -> Resistor_SMD:R_0603_1608Metric
- R10: value 2m -> 13k3; footprint WSLP25122L500FEA:RESC6432X89N -> Resistor_SMD:R_0603_1608Metric
- R11: value 10k -> 22k; footprint Resistor_SMD:R_0805_2012Metric -> Resistor_SMD:R_0603_1608Metric; moved to B.Cu
- R12: value 10k -> 100; footprint Resistor_SMD:R_0805_2012Metric -> Resistor_SMD:R_0603_1608Metric; moved to B.Cu
- R13: value 10k -> 1k; footprint Resistor_SMD:R_0805_2012Metric -> Resistor_SMD:R_0603_1608Metric; moved to B.Cu
- R14: value 10k -> 22k; footprint Resistor_SMD:R_0805_2012Metric -> Resistor_SMD:R_0603_1608Metric
- R16: renamed from R8; value 10k -> 4k7; footprint Resistor_SMD:R_0805_2012Metric -> Resistor_SMD:R_0603_1608Metric
- R17: renamed from R9; value 10k -> 4k7; footprint Resistor_SMD:R_0805_2012Metric -> Resistor_SMD:R_0603_1608Metric
- R19, R20: value 1k5 -> 4k7; footprint Resistor_SMD:R_0805_2012Metric -> Resistor_SMD:R_0603_1608Metric
- R2: value 47k -> 360k; footprint Resistor_SMD:R_0805_2012Metric -> Resistor_SMD:R_0603_1608Metric
- R22: renamed from R6; footprint Resistor_SMD:R_0805_2012Metric -> Resistor_SMD:R_0603_1608Metric
- R23, R24: value 220k -> 4k7; footprint Resistor_SMD:R_0805_2012Metric -> Resistor_SMD:R_0603_1608Metric
- R25, R27: footprint Resistor_SMD:R_0805_2012Metric -> Resistor_SMD:R_0603_1608Metric
- R26: renamed from R5; footprint Resistor_SMD:R_0805_2012Metric -> Resistor_SMD:R_0603_1608Metric
- R28: value 100k -> 4k7; footprint Resistor_SMD:R_0805_2012Metric -> Resistor_SMD:R_0603_1608Metric; moved to F.Cu
- R29: value 13k3 -> 4k7; footprint Resistor_SMD:R_0805_2012Metric -> Resistor_SMD:R_0603_1608Metric; moved to F.Cu
- R3: value 6k8 -> 220k; footprint Resistor_SMD:R_0805_2012Metric -> Resistor_SMD:R_0603_1608Metric
- R30: value 4k7 -> 6k8; footprint Resistor_SMD:R_0805_2012Metric -> Resistor_SMD:R_0603_1608Metric; moved to B.Cu
- R31: renamed from R15; footprint Resistor_SMD:R_0805_2012Metric -> Resistor_SMD:R_0603_1608Metric
- R32: value 22k -> 4k7; footprint Resistor_SMD:R_0805_2012Metric -> Resistor_SMD:R_0603_1608Metric
- R33: value 100 -> 4k7; footprint Resistor_SMD:R_0805_2012Metric -> Resistor_SMD:R_0603_1608Metric
- R35: renamed from R18; value 10k -> 4k7; footprint Resistor_SMD:R_0805_2012Metric -> Resistor_SMD:R_0603_1608Metric
- R39: value 360k -> 5m; footprint Resistor_SMD:R_0805_2012Metric -> footprints:RESC6432X89N; moved to B.Cu
- R40: value 10k -> 4k7; footprint Resistor_SMD:R_0805_2012Metric -> Resistor_SMD:R_0603_1608Metric; moved to B.Cu
- S2: value KMR211G_LFS -> ADTSM644KVTR; footprint KMR211G_LFS:KMR_2 -> footprints:ADTSM644KVTR; moved to F.Cu
- TP7: value 5V_TP -> VDD_TP
- TP8: value VDD_TP -> SW_TP; footprint TestPoint:TestPoint_THTPad_D1.0mm_Drill0.5mm -> TestPoint:TestPoint_Pad_D1.0mm
- TP9: value 3.3V_TP -> DIAG_TP; footprint TestPoint:TestPoint_THTPad_D1.0mm_Drill0.5mm -> TestPoint:TestPoint_Pad_D1.0mm
- U1: value PEC11L-4220F-S0015 -> ~; footprint PEC11L-4220F-S0015:PEC11L4220FS0015 -> footprints:Adafruit_240x320_TFT
- moved R39 126.8 mm to (186.5, 89.0), turned to 180 degrees
- moved IC4 121.4 mm to (185.2, 137.5), turned to 90 degrees
- moved R28 114.8 mm to (190.2, 139.8), turned to 0 degrees
- moved C32 112.6 mm to (196.0, 109.0), turned to 180 degrees
- moved R29 111.7 mm to (190.2, 136.8), turned to 0 degrees
- moved IC6 110.4 mm to (194.8, 131.8), turned to 90 degrees
- moved R40 109.3 mm to (169.2, 113.5)
- moved C13 109.0 mm to (196.2, 142.0)
- moved IC3 107.6 mm to (167.2, 75.5), turned to 90 degrees
- moved J4 106.4 mm to (168.6, 111.8), turned to -90 degrees
- moved J1 104.0 mm to (180.5, 146.2), turned to 180 degrees
- moved R16 103.8 mm to (195.2, 120.2)
- moved R26 103.4 mm to (196.7, 120.2)
- moved C26 102.4 mm to (181.5, 128.8), turned to 0 degrees
- moved H2 102.1 mm to (197.0, 147.0)
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- renumbered C4 to C35, C17 to C38, C18 to C39, IC1 to IC5
Connections:
- C10 pad 1: /ENC_A -> /TC
- C11 pad 1: Net-(IC2-VDDA) -> /Current
- C12 pad 1: Net-(IC2-VDDA) -> GND
- C12 pad 2: GND -> Net-(IC2-PF1/OSC_OUT)
- C13 pad 1: GND -> Net-(C13-Pad1)
- C13 pad 2: +5V -> /VDD_IN_USBCPD
- C14 pad 2: VDD -> /NRST
- C15 pad 1: /TC -> GND
- C15 pad 2: GND -> +5V
- C16 pad 1: /Current -> /VBUS
- C20 pad 1: /VBUS -> +3.3V
- C21 pad 1: GND -> +3.3V
- C21 pad 2: VDD -> GND
- C24 pad 1: Net-(IC6-BOOT) -> /VCCA
- C24 pad 2: Net-(IC6-SW) -> GND
- C25 pad 1: GND -> /VCCA
- C25 pad 2: +5V -> GND
- C26 pad 1: Net-(IC6-FB) -> /SW1
- C26 pad 2: +5V -> GND
- C27 pad 1: GND -> /SW2
- C27 pad 2: +5V -> GND
- C3 pad 1: Net-(C3-Pad1) -> Net-(IC2-PF0/OSC_IN)
- C32 pad 1: GND -> /Handle_sense1
- C32 pad 2: +5V -> GND
- C33 pad 1: Net-(IC7-VREG_1V2) -> /ENC_B
- C34 pad 1: /Handle_sense1 -> /ENC_A
- C35 pad 2: Net-(IC1-BOOST) -> Net-(IC5-TS)
- C5 pad 2: /VBUS -> VDD
- C6 pad 2: +5V -> VDD
- C7 pad 1: GND -> Net-(IC3-FB)
- C7 pad 2: /NRST -> +5V
- C8 pad 1: /SW1 -> GND
- C8 pad 2: GND -> +5V
- C9 pad 1: /ENC_B -> GND
- C9 pad 2: GND -> +5V
- D10 pad 1: Net-(D10-CATHODE_1) -> /RED
- D10 pad 2: Net-(D10-CATHODE_2) -> /BLUE
- D12 pad 1: GND -> /USB_D+
- D12 pad 2: +3.3V -> /USB_D-
- D12 pad 3: /VDD_inp -> GND
- D2 pad 1: Net-(IC1-BOOST) -> GND
- D2 pad 2: +5V -> +3.3V
- D5 pad 3: Net-(D6-common) -> /Handle_inp1
- D7 pad 1: /RED -> GND
- D7 pad 2: /BLUE -> +3.3V
- D9 pad 1: GND -> Net-(IC5-TS)
- D9 pad 2: /VDD_IN -> +5V
- IC2 pad 10: /SW1 -> /USR1
- IC2 pad 11: /ENC_B -> /Current
- IC2 pad 12: /SW_3 -> /TC
- IC2 pad 13: /VDD_inp -> /SPI_DC
- IC2 pad 14: GND -> /SPI_RST
- IC2 pad 15: Net-(IC2-VDDA) -> /SPI_SCK
- IC2 pad 16: GND -> /SPI_CS
- IC2 pad 17: +3.3V -> /SPI_MOSI
- IC2 pad 18: /Handle_inp2 -> /SD_CS
- IC2 pad 19: /Handle_inp1 -> GND
- IC2 pad 2: /SPI_DC -> /Buzzer
- IC2 pad 20: /Stand_inp -> GND
- IC2 pad 21: /USB_D- -> GND
- IC2 pad 22: /USB_D+ -> GND
- IC2 pad 23: /SWDIO -> GND
- IC2 pad 24: /SWCLK -> +3.3V
- IC2 pad 25: /SCL -> /Stand_inp
- IC2 pad 26: /SPI_SCK -> /VDD_inp
- IC2 pad 27: /SPI_RST -> /Handle_inp2
- IC2 pad 28: /SPI_MOSI -> /Handle_inp1
- IC2 pad 29: /SPI_CS -> /USR2
- IC2 pad 3: /SD_CS -> unconnected-(IC2-PC14/OSC32_IN-Pad3)
- IC2 pad 30: /SDA -> unconnected-(IC2-PA9-Pad30)
- IC2 pad 31: /Buzzer -> unconnected-(IC2-PA10-Pad31)
- IC2 pad 32: GND -> /USB_D-
- IC2 pad 4: /NRST -> unconnected-(IC2-PC15/OSC32_OUT-Pad4)
- IC2 pad 5: /TC -> Net-(IC2-PF0/OSC_IN)
- IC2 pad 6: /Current -> Net-(IC2-PF1/OSC_OUT)
- IC2 pad 7: /SW_2 -> /NRST
- IC2 pad 8: /Heater -> GND
- IC2 pad 9: /ENC_A -> /VCCA
- IC3 pad 1: /TC -> GND
- IC3 pad 2: Net-(IC3A--) -> Net-(IC3-SW)
- IC3 pad 3: Net-(IC3A-+) -> VDD
- IC3 pad 4: GND -> Net-(IC3-FB)
- IC3 pad 5: Net-(IC3B-+) -> unconnected-(IC3-EN-Pad5)
- IC3 pad 6: Net-(IC3B--) -> Net-(IC3-BOOT)
- IC4 pad 1: /Thermocouple_1 -> /CC1
- IC4 pad 2: Net-(IC4--IN_A) -> /CC1
- IC4 pad 3: Net-(IC4-+IN_A) -> (no net)
- IC4 pad 4: GND -> /CC2
- IC4 pad 5: Net-(IC4-+IN_B) -> /CC2
- IC4 pad 6: Net-(IC4--IN_B) -> GND
- IC4 pad 7: /Current_1 -> /SCL
- IC4 pad 8: +3.3V -> /SDA
- IC4 pad 9: GND -> Net-(IC4-DISCH)
- IC5 pad 6: Net-(IC1-BOOST) -> /RED
- IC5 pad 8: /RED -> Net-(IC5-TS)
- IC6 pad 1: GND -> Net-(IC6-GATE)
- IC6 pad 2: Net-(IC6-SW) -> /VDD_IN_USBCPD
- IC6 pad 3: VDD -> /VDD_IN_USBCPD
- IC6 pad 4: Net-(IC6-FB) -> /VDD_IN_USBCPD
- IC6 pad 5: unconnected-(IC6-EN-Pad5) -> GND
- IC6 pad 6: Net-(IC6-BOOT) -> (no net)
- J4 pad 1: /Stand_sense -> /BOOT0
- J4 pad 2: /Handle_sense2 -> +3.3V
- L1 pad 1: Net-(IC6-SW) -> Net-(IC3-SW)
- Q1 pad 4: /USB_PD_GATE -> Net-(Q1-G)
- Q1 pad 5: /VDD_IN -> /VDD_IN_USBCPD
- R1 pad 1: Net-(C3-Pad1) -> /RED
- R1 pad 2: /VDD_inp -> Net-(IC1A-+)
- R10 pad 1: /BLUE -> Net-(IC3-FB)
- R11 pad 1: /ENC_B -> Net-(Q1-G)
- R11 pad 2: +3.3V -> /VBUS
- R12 pad 1: +3.3V -> Net-(Q1-G)
- R12 pad 2: /SW1 -> Net-(C13-Pad1)
- R13 pad 1: +3.3V -> /VBUS
- R13 pad 2: /ENC_A -> Net-(IC4-VBUS_VS_DISCH)
- R14 pad 1: GND -> Net-(IC4-VBUS_EN_SNK)
- R14 pad 2: /Buzzer -> Net-(Q1-G)
- R19 pad 1: /GREEN -> /Handle_inp1
- R19 pad 2: Net-(IC3A--) -> /Handle_sense1
- R2 pad 1: VDD -> Net-(IC1A-+)
- R2 pad 2: Net-(C3-Pad1) -> GND
- R20 pad 1: /RED -> +5V
- R20 pad 2: Net-(IC3A-+) -> Net-(LS1--)
- R23 pad 1: Net-(IC3B-+) -> /SCL
- R23 pad 2: GND -> +3.3V
- R24 pad 1: /Current -> /SDA
- R24 pad 2: Net-(IC3B--) -> +3.3V
- R25 pad 1: /BLUE -> Net-(C29-Pad1)
- R25 pad 2: Net-(IC3B-+) -> /VDD_inp
- R27 pad 1: /SDA -> /SW1
- R27 pad 2: +3.3V -> GND
- R28 pad 1: +5V -> /SW2
- R28 pad 2: Net-(IC6-FB) -> GND
- R29 pad 1: Net-(IC6-FB) -> /SW3
- R3 pad 1: Net-(C3-Pad1) -> Net-(IC1B-+)
- R30 pad 1: /SCL -> Net-(C29-Pad1)
- R30 pad 2: +3.3V -> GND
- R32 pad 1: Net-(IC7-VBUS_EN_SNK) -> /ENC_B
- R32 pad 2: Net-(Q5-G) -> +3.3V
- R33 pad 1: Net-(Q5-G) -> +3.3V
- R33 pad 2: Net-(C31-Pad1) -> /ENC_A
- R39 pad 1: Net-(IC3A-+) -> /BLUE
- R40 pad 1: +3.3V -> /BOOT0
- R40 pad 2: /SW2 -> GND
- S2 pad 1: +3.3V -> /SW2
- S2 pad 2: /Buzzer -> +3.3V
- TP7 pad 1: +5V -> VDD
- TP8 pad 1: VDD -> /Heater
- TP9 pad 1: +3.3V -> /USR1
- U1 pad 1: /SW1 -> +5V
- U1 pad 2: GND -> unconnected-(U1-NC-Pad2)
- U1 pad 3: /ENC_B -> GND
- U1 pad 4: GND -> /SPI_SCK
- U1 pad 5: /ENC_A -> unconnected-(U1-NC-Pad5)
Routing:
- net GND: track 515.3 -> 600.5 mm, vias 98 -> 132
- net VDD: track 131.0 -> 56.9 mm, vias 4 -> 2
- net +3.3V: track 178.0 -> 231.8 mm, vias 15 -> 19
- net /SPI_CS: track 65.5 -> 14.1 mm, vias 4 -> 0
- net /SW3: track 0.00 -> 43.2 mm, vias 0 -> 1
- net Net-(J5-DN1): track 39.7 -> 0.00 mm
- net /SWCLK: track 18.3 -> 57.9 mm, vias 2 -> 4
- net Net-(Q2-Pad1): track 36.7 -> 0.00 mm, vias 1 -> 0
- net /VDD_IN: track 27.8 -> 64.2 mm, vias 0 -> 9
- net Net-(J5-DP1): track 35.9 -> 0.00 mm
- net /SCL: track 76.0 -> 40.5 mm, vias 5 -> 2
- net /SWDIO: track 15.6 -> 50.7 mm, vias 1 -> 3
- net /SW2: track 0.00 -> 31.8 mm, vias 0 -> 1
- net /Thermocouple_1: track 30.8 -> 0.00 mm
- net /Current: track 0.00 -> 28.4 mm, vias 0 -> 2
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- added copper zone on B.Cu, net /VBUS
- added copper zone on B.Cu, net /VDD_IN_USBCPD
- removed copper zone on B.Cu, net +5V
- removed copper zone on F.Cu, net +5V
- removed copper zone on F.Cu, net /RED
- removed copper zone on F.Cu, net /VDD_IN
Other:
- board size 39 x 71 mm -> 39 x 82.5 mm
- board text added: "2025-01"
- board text added: "9-24 V"
- board text added: "<---- SCREEN SUPPORT ---->"
- board text added: "AxxSolder"
- board text added: "BLU"
- board text added: "BOOT0"
- board text added: "GRN"
- board text added: "IN1"
- board text added: "IN2"
- board text added: "Input Voltage"
- board text added: "SCL"
- board text added: "SDA"
- board text added: "STND"
- board text added: "STUSB4500"
- board text added: "SW"
- board text added: "USBC-PD 100W"
- board text added: "USR1"
- board text added: "USR2"
- board text added: "V3.0"
- board text added: "V_IN"
- board text removed: "+"
- board text removed: "-"
- board text removed: "3.3"
- board text removed: "AxxSolder V3.0"
- board text removed: "BLUE"
- board text removed: "BOOT"
- board text removed: "CLK"
- board text removed: "DIO"
- board text removed: "GREEN"
- board text removed: "HANDLE"
- board text removed: "Input: 9-24 V"
- board text removed: "RST"
- board text removed: "STAND"
- board text removed: "SWD"
- board text removed: "TX"
- board text removed: "USBC_DN"
- board text removed: "USBC_DP"
- board text removed: "VDD+"
