File: AxxSolder.kicad_sch (KiCad schematic)
At the start: 113 parts, among them IC1 LTC4440AHMS8E-5#PBF, IC2 STM32G431KBT6, IC4 OPA2333AIDRBR, IC5 STM32G431KBT6, IC6 TPS54302DDCR, IC7 STUSB4500QTR, IC8 USBLC6-2P6, J1 Conn_01x07_Male, J2 USB_B_Micro, J5 USB4105-GF-A-120, J6 Conn_01x06_Socket, Q1 STL9P3LLH6, Q2 2N7002NXAKR, U1 PEC11L-4220F-S0015, U2 BSC014N04LS

Commit message: update filestructure for AxxSolder V3.0 and forward
Parts:
- removed D10: ESDA25W, ESDA25W:SOT65P210X110-3N, symbol ESDA25W:ESDA25W
- removed D11: 1N5819HW-7-F, 1N5819HW-7-F:SOD3716X145N, symbol 1N5819HW-7-F:1N5819HW-7-F
- removed D13: V7NM103-M3_I, V7NM103-M3_I:V7NM103M3I, symbol V7NM103-M3_I:V7NM103-M3_I
- removed D4: Waveshare 1.5inch OLED Module, 1_5inch-rgb-oled-module_asm-1110:1_5inch-rgb-oled-module_asm-1110, symbol 1_5inch-rgb-oled-module_asm-1110:1_5inch-rgb-oled-module_asm-1110
- removed D5, D6: BAT54S, BAT54S,215:SOT95P230X110-3N, symbol Device:D_Schottky_Dual_Series_AKC
- removed D9: SMBJ24CA, SMBJ24CA:DIOM5436X261N, symbol SMBJ24CA:SMBJ24CA
- removed IC4: OPA2333AIDRBR, OPA2333AIDRBR:SON65P300X300X100-9N-D, symbol OPA2333AIDRBR:OPA2333AIDRBR
- removed IC8: USBLC6-2P6, USBLC6-2P6:USBLC62P6, symbol USBLC6-2P6:USBLC6-2P6
- removed J1: Conn_01x07_Male, 691243310007:691243310007, symbol Connector:Conn_01x07_Male
- removed J2: USB_B_Micro, USB3140-30-0230-1-C_REVE1:GCT_USB3140-30-0230-1-C_REVE1, symbol Connector:USB_B_Micro
- removed J5: USB4105-GF-A-120, USB4105-GF-A:GCT_USB4105-GF-A-120, symbol USB4105-GF-A-120:USB4105-GF-A-120
- removed J6: Conn_01x06_Socket, Connector_PinSocket_2.54mm:PinSocket_1x06_P2.54mm_Vertical, symbol Connector:Conn_01x06_Socket
- removed JP1, JP2: SolderJumper_2_Open, Jumper:SolderJumper-2_P1.3mm_Open_TrianglePad1.0x1.5mm, symbol Jumper:SolderJumper_2_Open
- removed Q1: STL9P3LLH6, STL9P3LLH6:STL20N6F7, symbol STL9P3LLH6:STL9P3LLH6
- removed S2: KMR211G_LFS, KMR211G_LFS:KMR_2, symbol KMR211G_LFS:KMR211G_LFS
- added C32: 10u, Capacitor_SMD:C_0805_2012Metric, symbol Device:C_Small
- added C33: 1u, Capacitor_SMD:C_0805_2012Metric, symbol Device:C_Small
- added C34, C35, C36, C37: 100n, Capacitor_SMD:C_0805_2012Metric, symbol Device:C_Small
- added D11, D5: BAV199WQ-7, Library:SOT65P210X110-3N, symbol BAV199WQ-7:BAV199WQ-7
- added D4: SMBJ24A, DIOM5436X261N, symbol SMBJ24A:SMBJ24A
- added D6: ESDA25W, SOT65P210X110-3N, symbol ESDA25W:ESDA25W
- added D9: BAT54S, BAT54S,215:SOT95P230X110-3N, symbol Device:D_Schottky_Dual_Series_AKC
- added FB1: BLM18HE601SN1D, footprints:BLM18SP221SN1B, symbol BLM18HE601SN1D:BLM18HE601SN1D
- added IC3: OPA2387DSGT, SON50P200X200X80-9N, symbol OPA2387DSGT:OPA2387DSGT
- added J2: Conn_01x05_Socket, symbol Connector:Conn_01x05_Socket
- added J3: USB_C_Receptacle_USBC, symbol Connector:USB_C_Receptacle_USB2.0
- added J4: 691243110008, footprints:691243110008, symbol 691243110008:691243110008
- added Q5: STL9P3LLH6, STL20N6F7, symbol STL9P3LLH6:STL9P3LLH6
- added R36: 1k, Resistor_SMD:R_0805_2012Metric, symbol Device:R_Small
- added R37: 4k7, Resistor_SMD:R_0805_2012Metric, symbol Device:R_Small
- added R38: 22k, Resistor_SMD:R_0805_2012Metric, symbol Device:R_Small
- added R39: 360k, Resistor_SMD:R_0805_2012Metric, symbol Device:R_Small
- added R40, R41: 10k, Resistor_SMD:R_0805_2012Metric, symbol Device:R_Small
- added SW1, SW2, SW3, SW4: SW_Push, symbol Switch:SW_Push
- added TC3: TC, symbol Device:Thermocouple
- added U3: TPD2E2U06QDBZRQ1, SOT95P237X95-3N, symbol TPD2E2U06QDBZRQ1:TPD2E2U06QDBZRQ1
- added U4: ~, symbol Adafruit_240x320_TFT:Adafruit_240x320_TFT
- C5: value 10u -> 4.7u
- D8: value ESDA25P35-1U1M -> ESDA25P35; footprint ESDA25P35-1U1M:ESDA25P351U1M -> ESDA25P351U1M
- IC1: value LTC4440AHMS8E-5#PBF -> LTC4440AHMS8E; footprint LTC4440AHMS8E-5#PBF:SOP65P490X110-9N -> SOP65P490X110-9N
- IC7: footprint STUSB4500QTR:QFN50P400X400X100-25N-D -> QFN50P400X400X100-25N-D
- L1: value SRP7028CC-100M -> SRP7028CC; Mouser Part Number (none) -> e
- Q2: footprint 2N7002NXAKR:SOT95P230X110-3N -> SOT95P230X110-3N
- R21: value 470k -> 10k; Manufacturer_Part_Number ERJ-6ENF4703V -> ERJ-6ENF1002V
- R22: value 470k -> 360k
- R31: value 1k -> Heater; footprint Resistor_SMD:R_0805_2012Metric -> (none); Assembly Comment (none) -> N/A; Manufacturer_Name Panasonic -> (none); Manufacturer_Part_Number ERJ-6ENF1001V -> (none); now left out of the parts list
- R33: value 100k -> 100
- R34: value 22k -> 10k; Manufacturer_Part_Number ERJ-6ENF2202V -> ERJ-6ENF1002V
- TP5: value Thermocouple_TP -> TC_TP
Connections:
- net Thermocouple_2 is gone; now on net SW1: IC2.10 (PA5), IC5.10 (PA5)
- net +3.3V: now also R21.1, R34.1, D11.2, D5.2, D9.2 (K), FB1.2, IC3.8 (V+), J2.2 (Pin_2), R40.1, R41.1, SW4.1; no longer C11.1, C12.1, IC2.15 (VDDA), IC5.15 (VDDA)
- net +5V: now also TP8.1, C32.2, U4.1 (VIN)
- net BLUE: now also R25.1, J4.5; no longer R25.2
- net Buzzer: now also SW4.2
- net GND: now also R26.2, C32.1, C33.2, C34.2, C35.2, C36.2, C37.2, D11.1, D4.2 (A), D5.1, D6.3, D9.1 (A), IC3.4 (V-), IC3.9 (THERMAL_PAD), J2.1 (Pin_1), J3.A1 (GND), J3.A12 (GND), J3.B1 (GND), J3.B12 (GND), J3.S1 (SHIELD), J4.7, R39.2, SW1.1, SW2.1, SW3.1, U3.3 (GND), U4.3 (GND); no longer R21.2, R26.1
- net GREEN: now also J4.4
- net NRST: now also J2.3 (Pin_3)
- net RED: now also J4.6
- net SCL: now also R30.1; no longer R27.1
- net SDA: now also R27.1; no longer R30.1
- net SPI_DC: now also U4.9 (DC)
- net SPI_MOSI: now also U4.6 (MOSI)
- net SPI_RST: now also U4.8 (RST)
- net SPI_SCK: now also U4.4 (SCK)
- net SWCLK: now also J2.4 (Pin_4), J3.A8 (SBU1)
- net SWDIO: now also J2.5 (Pin_5), J3.B8 (SBU2)
- net Stand_inp: no longer C29.1
- net Stand_sense: now also C29.1, J4.1
- net USB_D+: now also J3.A6 (D+), J3.B6 (D+), U3.1 (IO1)
- net USB_D-: now also J3.A7 (D-), J3.B7 (D-), U3.2 (IO2)
- net VBUS: now also C20.1, J3.A4 (VBUS), J3.A9 (VBUS), J3.B4 (VBUS), J3.B9 (VBUS), Q5.1 (S), R36.1, R38.2; no longer R31.2, R33.2
- net VDD: now also D4.1 (K); no longer C31.2, R35.2, TP8.1
- net VDD_IN: now also C31.2, R35.1, J4.8, Q5.5 (D)
- net at C30.1: now also IC7.23 (VREG_2V7); no longer IC7.21 (VREG_1V2)
- net at R19.2, R22.2: now also D5.3, IC3.2 (-)
- net at R20.2: now also D11.3, IC3.3 (+), R39.1; no longer R21.1
- net Current: now reaches R24.1
- net Current: now also C16.1, IC2.6 (PA1), IC5.6 (PA1), TP6.1, IC3.7; no longer R26.2
- net CC2: now reaches IC7.4 (CC2), IC7.5 (CC2DB)
- net CC2: now also D6.1, J3.B5 (CC2)
- net CC1: now reaches IC7.1 (CC1DB), IC7.2 (CC1)
- net CC1: now also D6.2, J3.A5 (CC1)
- net at C31.1: now also R33.2; no longer R34.2
- net at R23.1: now also R25.2, IC3.5 (+); no longer R25.1
- net at IC7.9 (DISCH): now also R35.2; no longer R35.1
- net at IC7.18 (VBUS_VS_DISCH): now also R36.2; no longer R31.1
- net Busvoltage renamed VDD_inp
- removed net Current_1: C16.1, IC2.6 (PA1), IC5.6 (PA1), R24.2, TP6.1
- net Current_2 renamed SW_3
- net ENC_Button renamed SW1
- net SW1: now also C35.1, R41.2, SW1.2; no longer IC2.29 (PB6), IC5.29 (PB6)
- net HEATER_2 renamed Handle_inp2
- net Handle_inp2: now also D3.3 (common), R6.1
- removed net Handle_inp: C28.1, D3.3 (common), IC2.19 (PA9), IC5.19 (PA9), R6.1
- net Handle_sense renamed Handle_sense2
- net Handle_sense2: now also C28.1, J4.2
- net Heater_1 renamed Heater
- net Identification_inp renamed SD_CS
- net SD_CS: now also U4.10 (SDCS)
- net MCU_TX renamed SW_2
- net Thermocouple_1 renamed TC
- net TC: now also IC3.1
- net USB_PD_GATE: no longer names the net of R32.2, R33.1
- net USB_PD_GATE: now also Q5.4 (G), R38.1; no longer R34.1
- new net: R31.2, TC3.1 (+)
- new net: IC3.6 (-), R24.2, R26.1
- new net: C11.1, C12.1, FB1.1, IC2.15 (VDDA), IC5.15 (VDDA)
- new net: C33.1, IC7.21 (VREG_1V2)
- new net Handle_inp1: D9.3 (common), IC2.19 (PA9), IC5.19 (PA9), R37.1
- new net Handle_sense1: C34.1, J4.3, R34.2, R37.2
- new net SPI_CS: IC2.29 (PB6), IC5.29 (PB6), U4.7 (CS)
- new net SW2: C36.1, R40.2, SW2.2
- new net SW3: C37.1, R21.2, SW3.2
Other:
- note added: "(and 6 for C210)"
- note added: "2023-12-06"
- note added: "240x320 TFT DISPLAY"
- note added: "3.3V LDO REGULATOR"
- note added: "5V SWITCHING VOLTAGE REGULATOR"
- note added: "A"
- note added: "AxxSolder"
- note added: "BLUE-pin 5"
- note added: "C115"
- note added: "GAIN: 240"
- note added: "GAIN: 46.8"
- note added: "GREEN-pin 1"
- note added: "I2C PULL-UPS"
- note added: "INPUTS"
- note added: "RED-pin 2"
- note added: "SCREW TERMINAL"
- note added: "USB C - Power Delivery"
- note added: "USER BUTTONS"
- note added: "VDD VOLTAGE SENSING"
- note removed: "3.3V Voltage Regulator"
- note removed: "BLUE - pin 5 (and 6 for C210)"
- note removed: "DC/DC VDD to 5V"
- note removed: "Firmware update USB"
- note removed: "GREEN - pin 1"
- note removed: "INPUT VOLTAGE SENSING"
- note removed: "INPUTS FROM SOLDERING STATION"
- note removed: "MAIN SCREW TERMINAL"
- note removed: "OLED DISPLAY"
- note removed: "RED - pin 2"
- moved on the sheet: C1, C10, C11, C12, C13, C14, C15, C16, C17, C18, C19, C2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

Commit message: multiple updates for AxxSolder hw 3.0
Parts:
- removed C11, C7, C8: 100n, Capacitor_SMD:C_0805_2012Metric, symbol Device:C_Small
- removed C23: 330u, EMZR500ARA331MJA0G:CAPAE1030X1050N, symbol EMZR500ARA331MJA0G:EMZR500ARA331MJA0G
- removed C5: 4.7u, Capacitor_SMD:C_0805_2012Metric, symbol Device:C_Small
- removed C6: 10u, Capacitor_SMD:C_0805_2012Metric, symbol Device:C_Small
- removed D8: ESDA25P35, ESDA25P351U1M, symbol ESDA25P35-1U1M:ESDA25P35-1U1M
- removed H3, H4: MountingHole, MountingHole:MountingHole_3mm, symbol Mechanical:MountingHole
- removed IC2: STM32G431KBT6, STM32G431KBT6:QFP80P900X900X160-32N, symbol STM32G431KBT6:STM32G431KBT6
- removed IC5: STM32G431KBT6, Package_DFN_QFN:UFQFPN-32-1EP_5x5mm_P0.5mm_EP3.5x3.5mm, symbol STM32G431KBT6:STM32G431KBT6
- removed J3: USB_C_Receptacle_USBC, symbol Connector:USB_C_Receptacle_USB2.0
- removed J4: 691243110008, footprints:691243110008, symbol 691243110008:691243110008
- removed R10: 2m, WSLP25122L500FEA:RESC6432X89N, symbol Device:R_Small
- removed R12, R14: 10k, Resistor_SMD:R_0805_2012Metric, symbol Device:R_Small
- removed SW1, SW2, SW3, SW4: SW_Push, symbol Switch:SW_Push
- removed U1: PEC11L-4220F-S0015, PEC11L-4220F-S0015:PEC11L4220FS0015, symbol PEC11L-4220F-S0015:PEC11L-4220F-S0015
- removed U4: ~, symbol Adafruit_240x320_TFT:Adafruit_240x320_TFT
- added C14, C20, C21, C24: 100n, Capacitor_SMD:C_0603_1608Metric, symbol Device:C_Small
- added C19, C25: 10u, Capacitor_SMD:C_0603_1608Metric, symbol Device:C_Small
- added C3: 10p, Capacitor_SMD:C_0603_1608Metric, symbol Device:C_Small
- added D11: ESDA25P35, footprints:ESDA25P351U1M, symbol ESDA25P35-1U1M:ESDA25P35-1U1M
- added IC2: STM32F303CCT6TR, footprints:QFP50P900X900X160-48N, symbol STM32F303CCT6TR:STM32F303CCT6TR
- added IC6: MAX16171ATA_VY+T, SON50P300X200X80-9N, symbol MAX16171ATA_VY+T:MAX16171ATA_VY+T
- added J1: USB4110-GF-A, footprints:USB4110GFA, symbol USB4110-GF-A:USB4110-GF-A
- added J2: 691243110009, footprints:691243110009, symbol 691243110009:691243110009
- added J4: Conn_01x02_Pin, Connector_PinHeader_1.27mm:PinHeader_1x02_P1.27mm_Vertical, symbol Connector:Conn_01x02_Pin
- added Q3: STL10N3LLH5, STL10N3LLH5, symbol STL10N3LLH5:STL10N3LLH5
- added R39: 5m, footprints:RESC6432X89N, symbol WSLP25125L000FEA:WSLP25125L000FEA
- added R40: 4k7, Resistor_SMD:R_0603_1608Metric, symbol Device:R_Small
- added S1, S2, S3: ADTSM644KVTR, footprints:ADTSM644KVTR, symbol ADTSM644KVTR:ADTSM644KVTR
- added TP10, TP11, TP12, TP9: DIAG_TP, TestPoint:TestPoint_Pad_D1.0mm, symbol Connector:TestPoint
- added TP7: VDD_TP, TestPoint:TestPoint_THTPad_D1.0mm_Drill0.5mm, symbol Connector:TestPoint
- added TP8: SW_TP, TestPoint:TestPoint_Pad_D1.0mm, symbol Connector:TestPoint
- added U1: ~, footprints:Adafruit_240x320_TFT, symbol Adafruit_240x320_TFT:Adafruit_240x320_TFT
- added U3: PEC11J-9220F-S0015, footprints:PEC11J9220FS0015, symbol PEC11J-9220F-S0015:PEC11J-9220F-S0015
- added Y1: NX2016SA-32M-EXS00A-CS06465, footprints:NX2016SA32MEXS00ACS06465, symbol NX2016SA-32M-EXS00A-CS06465:NX2016SA-32M-EXS00A-CS06465
- C1: renamed from C13; footprint Capacitor_SMD:C_0805_2012Metric -> Capacitor_SMD:C_0603_1608Metric
- C10: renamed from C15; footprint Capacitor_SMD:C_0805_2012Metric -> Capacitor_SMD:C_0603_1608Metric
- C11: renamed from C16; footprint Capacitor_SMD:C_0805_2012Metric -> Capacitor_SMD:C_0603_1608Metric
- C12: value 10u -> 10p; footprint Capacitor_SMD:C_0805_2012Metric -> Capacitor_SMD:C_0603_1608Metric; Manufacturer_Part_Number GRM21BR6YA106ME43L -> GRM21A5C2E750FW01D
- C13: renamed from C31; footprint Capacitor_SMD:C_0805_2012Metric -> Capacitor_SMD:C_0603_1608Metric
- C15: renamed from C32; footprint Capacitor_SMD:C_0805_2012Metric -> Capacitor_SMD:C_0603_1608Metric
- C16: renamed from C20; footprint Capacitor_SMD:C_0805_2012Metric -> Capacitor_SMD:C_0603_1608Metric
- C17: renamed from C30; footprint Capacitor_SMD:C_0805_2012Metric -> Capacitor_SMD:C_0603_1608Metric
- C18: renamed from C33; footprint Capacitor_SMD:C_0805_2012Metric -> Capacitor_SMD:C_0603_1608Metric
- C2: renamed from C19; footprint Capacitor_SMD:C_0805_2012Metric -> Capacitor_SMD:C_0603_1608Metric
- C22: footprint Capacitor_SMD:C_0805_2012Metric -> Capacitor_SMD:C_0603_1608Metric
- C26: renamed from C35; footprint Capacitor_SMD:C_0805_2012Metric -> Capacitor_SMD:C_0603_1608Metric
- C27: renamed from C36; footprint Capacitor_SMD:C_0805_2012Metric -> Capacitor_SMD:C_0603_1608Metric
- C28: renamed from C37; footprint Capacitor_SMD:C_0805_2012Metric -> Capacitor_SMD:C_0603_1608Metric
- C29: renamed from C3; footprint Capacitor_SMD:C_0805_2012Metric -> Capacitor_SMD:C_0603_1608Metric
- C30: renamed from C29; footprint Capacitor_SMD:C_0805_2012Metric -> Capacitor_SMD:C_0603_1608Metric
- C31: renamed from C28; footprint Capacitor_SMD:C_0805_2012Metric -> Capacitor_SMD:C_0603_1608Metric
- C32: renamed from C34; footprint Capacitor_SMD:C_0805_2012Metric -> Capacitor_SMD:C_0603_1608Metric
- C33: renamed from C9; footprint Capacitor_SMD:C_0805_2012Metric -> Capacitor_SMD:C_0603_1608Metric
- C34: renamed from C10; footprint Capacitor_SMD:C_0805_2012Metric -> Capacitor_SMD:C_0603_1608Metric
- C36: renamed from C1; footprint Capacitor_SMD:C_0805_2012Metric -> Capacitor_SMD:C_0603_1608Metric
- C37: renamed from C2; footprint Capacitor_SMD:C_0805_2012Metric -> Capacitor_SMD:C_0603_1608Metric
- C4: renamed from C24; footprint Capacitor_SMD:C_0805_2012Metric -> Capacitor_SMD:C_0603_1608Metric
- C5: renamed from C21; footprint Capacitor_SMD:C_0805_2012Metric -> Capacitor_SMD:C_0603_1608Metric
- C6: renamed from C14; footprint Capacitor_SMD:C_0805_2012Metric -> Capacitor_SMD:C_0603_1608Metric
- C7: renamed from C26; footprint Capacitor_SMD:C_0805_2012Metric -> Capacitor_SMD:C_0603_1608Metric
- D1: renamed from D11; footprint Library:SOT65P210X110-3N -> footprints:SOT65P210X110-3N
- D10: renamed from D7; footprint PMEG10030ELPX:SODFL4725X110N -> footprints:SODFL4725X110N
- D12: renamed from U3; value TPD2E2U06QDBZRQ1 -> TPD2E2U06; footprint SOT95P237X95-3N -> footprints:SOT95P237X95-3N
- D2: renamed from D5; footprint Library:SOT65P210X110-3N -> footprints:SOT65P210X110-3N
- D3: renamed from D6; footprint SOT65P210X110-3N -> footprints:SOT65P210X110-3N
- D4: footprint DIOM5436X261N -> footprints:DIOM5436X261N
- D5: renamed from D9; footprint BAT54S,215:SOT95P230X110-3N -> footprints:SOT95P230X110-3N
- D6: renamed from D3; footprint BAT54S,215:SOT95P230X110-3N -> footprints:SOT95P230X110-3N
- D7: renamed from D12; footprint BAT54S,215:SOT95P230X110-3N -> footprints:SOT95P230X110-3N
- D8: renamed from D1; footprint BAT54S,215:SOT95P230X110-3N -> footprints:SOT95P230X110-3N
- D9: renamed from D2; footprint PMEG6020ER,115:PMEG6020ER115 -> footprints:PMEG6020ER115
- F1: renamed from F2; footprint 0154007:0154100DR -> footprints:0154100DR
- FB1: footprint footprints:BLM18SP221SN1B -> Resistor_SMD:R_0603_1608Metric
- H1, H2: footprint MountingHole:MountingHole_3mm -> MountingHole:MountingHole_2.5mm
- IC1: renamed from IC3; footprint SON50P200X200X80-9N -> footprints:SON50P200X200X80-9N
- IC3: renamed from IC6; footprint TPS54302DDCR:SOT95P280X110-6N -> footprints:SOT95P280X110-6N
- IC4: renamed from IC7; footprint QFN50P400X400X100-25N-D -> footprints:QFN50P400X400X100-25N-D
- IC5: renamed from IC1; footprint SOP65P490X110-9N -> footprints:SOP65P490X110-9N
- J3: renamed from J2; footprint (none) -> Connector_PinSocket_2.54mm:PinSocket_1x05_P2.54mm_Vertical
- L1: footprint SRP7028CC-100M:INDPM7366X300N -> footprints:INDPM7366X300N
- LS1: footprint CMI-9653S-SMT-TR:CMI9653SSMTTR -> footprints:CMI9653SSMTTR
- PS1: footprint LD1117AS33TR:SOT230P700X190-4N -> footprints:SOT230P700X190-4N
- Q1: renamed from Q5; footprint STL20N6F7 -> footprints:STL20N6F7
- Q2: footprint SOT95P230X110-3N -> footprints:SOT95P230X110-3N
- R1: renamed from R20; footprint Resistor_SMD:R_0805_2012Metric -> Resistor_SMD:R_0603_1608Metric
- R10: renamed from R29; footprint Resistor_SMD:R_0805_2012Metric -> Resistor_SMD:R_0603_1608Metric
- R11: renamed from R38; footprint Resistor_SMD:R_0805_2012Metric -> Resistor_SMD:R_0603_1608Metric
- R12: renamed from R33; footprint Resistor_SMD:R_0805_2012Metric -> Resistor_SMD:R_0603_1608Metric
- R13: renamed from R36; footprint Resistor_SMD:R_0805_2012Metric -> Resistor_SMD:R_0603_1608Metric
- R14: renamed from R32; footprint Resistor_SMD:R_0805_2012Metric -> Resistor_SMD:R_0603_1608Metric
- R15: renamed from R35; footprint Resistor_SMD:R_0805_2012Metric -> Resistor_SMD:R_0603_1608Metric
- R16: renamed from R8; value 10k -> 4k7; footprint Resistor_SMD:R_0805_2012Metric -> Resistor_SMD:R_0603_1608Metric
- R17: renamed from R9; value 10k -> 4k7; footprint Resistor_SMD:R_0805_2012Metric -> Resistor_SMD:R_0603_1608Metric
- R18: renamed from R34; value 10k -> 4k7; footprint Resistor_SMD:R_0805_2012Metric -> Resistor_SMD:R_0603_1608Metric
- R19: renamed from R37; footprint Resistor_SMD:R_0805_2012Metric -> Resistor_SMD:R_0603_1608Metric
- R2: renamed from R39; footprint Resistor_SMD:R_0805_2012Metric -> Resistor_SMD:R_0603_1608Metric
- R20: renamed from R17; footprint Resistor_SMD:R_0805_2012Metric -> Resistor_SMD:R_0603_1608Metric
- R21: renamed from R2; footprint Resistor_SMD:R_0805_2012Metric -> Resistor_SMD:R_0603_1608Metric
- R22: renamed from R6; footprint Resistor_SMD:R_0805_2012Metric -> Resistor_SMD:R_0603_1608Metric
- R23: renamed from R30; footprint Resistor_SMD:R_0805_2012Metric -> Resistor_SMD:R_0603_1608Metric
- R24: renamed from R27; footprint Resistor_SMD:R_0805_2012Metric -> Resistor_SMD:R_0603_1608Metric
- R25: renamed from R1; footprint Resistor_SMD:R_0805_2012Metric -> Resistor_SMD:R_0603_1608Metric
- R26: renamed from R5; footprint Resistor_SMD:R_0805_2012Metric -> Resistor_SMD:R_0603_1608Metric
- R27: renamed from R41; value 10k -> 4k7; footprint Resistor_SMD:R_0805_2012Metric -> Resistor_SMD:R_0603_1608Metric
- R28: renamed from R40; value 10k -> 4k7; footprint Resistor_SMD:R_0805_2012Metric -> Resistor_SMD:R_0603_1608Metric
- R29: renamed from R21; value 10k -> 4k7; footprint Resistor_SMD:R_0805_2012Metric -> Resistor_SMD:R_0603_1608Metric
- R3: renamed from R23; footprint Resistor_SMD:R_0805_2012Metric -> Resistor_SMD:R_0603_1608Metric
- R30: renamed from R3; footprint Resistor_SMD:R_0805_2012Metric -> Resistor_SMD:R_0603_1608Metric
- R31: renamed from R15; footprint Resistor_SMD:R_0805_2012Metric -> Resistor_SMD:R_0603_1608Metric
- R32: renamed from R11; value 10k -> 4k7; footprint Resistor_SMD:R_0805_2012Metric -> Resistor_SMD:R_0603_1608Metric
- R33: renamed from R13; value 10k -> 4k7; footprint Resistor_SMD:R_0805_2012Metric -> Resistor_SMD:R_0603_1608Metric
- R34: renamed from R16; value 10k -> 4k7; footprint Resistor_SMD:R_0805_2012Metric -> Resistor_SMD:R_0603_1608Metric
- R35: renamed from R18; value 10k -> 4k7; footprint Resistor_SMD:R_0805_2012Metric -> Resistor_SMD:R_0603_1608Metric
- R4: renamed from R25; footprint Resistor_SMD:R_0805_2012Metric -> Resistor_SMD:R_0603_1608Metric
- R5: renamed from R19; footprint Resistor_SMD:R_0805_2012Metric -> Resistor_SMD:R_0603_1608Metric
- R6: renamed from R28; footprint Resistor_SMD:R_0805_2012Metric -> Resistor_SMD:R_0603_1608Metric
- R7: renamed from R26; footprint Resistor_SMD:R_0805_2012Metric -> Resistor_SMD:R_0603_1608Metric
- R8: renamed from R22; footprint Resistor_SMD:R_0805_2012Metric -> Resistor_SMD:R_0603_1608Metric
- R9: renamed from R24; footprint Resistor_SMD:R_0805_2012Metric -> Resistor_SMD:R_0603_1608Metric
- U4: renamed from U2; footprint BSC014N04LS:BSC014N04LS -> footprints:BSC014N04LS
- renumbered C4 to C35, C17 to C38, C18 to C39, C25 to C8, C27 to C9, R31 to R36, R4 to R37, R7 to R38, TC3 to TC1, TC1 to TC2, TC2 to TC3, TP8 to TP1, TP9 to TP2, TP7 to TP3, TP6 to TP4, TP3 to TP6
Connections:
- net +3.3V: now also C20.1, C21.1, IC2.1 (VBAT), IC2.24 (VDD_1), IC2.36 (VDD_2), IC2.48 (VDD_3), J4.2 (Pin_2), S1.2, S2.2, S3.2, U3.D1; no longer R27.1, R28.1, R29.1
- net +5V: now also U1.1 (VIN)
- net BLUE: now also J2.6, R39.1
- net Buzzer: now also IC2.2 (PC13)
- net CC1: now also J1.A5 (CC1)
- net CC2: now also J1.B5 (CC2)
- net Current: now also IC2.11 (PA1)
- net ENC_A: now also IC2.39 (PB3), U3.C1
- net ENC_B: now also IC2.38 (PA15), U3.A1
- net GND: now also C12.1, R27.2, R28.2, R29.2, C14.1, C19.1, C20.2, C21.2, C24.2, C25.2, C3.2, D11.2 (A), IC2.19 (PB1), IC2.20 (PB2), IC2.21 (PB10), IC2.22 (PB11), IC2.23 (VSS_1), IC2.35 (VSS_2), IC2.47 (VSS_3), IC2.8 (VSSA/VREF-), IC6.5 (GND), IC6.9 (EP), J1.A1 (GND), J1.A12 (GND), J1.B1 (GND), J1.B12 (GND), J1.S1 (SHIELD), J2.8, R39.2, R40.2, U1.3 (GND), U3.B1, U3.MP, Y1.2; no longer C12.2
- net GREEN: now also J2.4, J2.5
- net Handle_inp1: now also IC2.28 (PB15)
- net Handle_inp2: now also IC2.27 (PB14)
- net Handle_sense1: now also J2.3
- net Handle_sense2: now also J2.2
- net Heater: now also IC2.43 (PB7), TP8.1
- net NRST: now also C14.2, IC2.7 (NRST)
- net RED: now also IC5.6 (BOOST), J2.7; no longer IC5.8 (TS)
- net SCL: now also IC2.45 (PB8), TP11.1
- net SDA: now also IC2.46 (PB9), TP12.1
- net SD_CS: now also IC2.18 (PB0), U1.10 (SDCS)
- net SPI_CS: now also IC2.16 (PA6), U1.7 (CS)
- net SPI_DC: now also IC2.13 (PA3), U1.9 (DC)
- net SPI_MOSI: now also IC2.17 (PA7), U1.6 (MOSI)
- net SPI_RST: now also IC2.14 (PA4), U1.8 (RST)
- net SPI_SCK: now also IC2.15 (PA5), U1.4 (SCK)
- net SW1: now also R27.1, IC2.40 (PB4), S1.1, U3.E1; no longer R27.2
- net SW2: now also R28.1, IC2.41 (PB5), S2.1; no longer R28.2
- net SW3: now also R29.1, IC2.42 (PB6), S3.1; no longer R29.2
- net SWCLK: now also IC2.37 (PA14), J1.A8 (SBU1)
- net SWDIO: now also IC2.34 (PA13), J1.B8 (SBU2)
- net Stand_inp: now also IC2.25 (PB12)
- net Stand_sense: now also J2.1
- net TC: now also IC2.12 (PA2)
- net USB_D+: now also IC2.33 (PA12), J1.A6 (D+), J1.B6 (D+)
- net USB_D-: now also IC2.32 (PA11), J1.A7 (D-), J1.B7 (D-)
- net VBUS: now also C19.2, D11.1 (K), J1.A4 (VBUS), J1.A9 (VBUS), J1.B4 (VBUS), J1.B9 (VBUS)
- net VDD: now also TP7.1
- net VDD_IN: now also IC6.8 (OUT), J2.9, Q3.5 (D); no longer C13.2, Q1.5 (D), R15.1
- net VDD_inp: now also IC2.26 (PB13)
- net VCCA: now reaches FB1.1
- net VCCA: now also C24.1, C25.1, IC2.9 (VDDA); no longer C12.1
- net at C35.2, D9.1: now also IC5.8 (TS); no longer IC5.6 (BOOST)
- new net: IC6.1 (GATE), Q3.4 (G)
- new net: C12.2, IC2.6 (PF1/OSC_OUT), Y1.3
- new net: C3.1, IC2.5 (PF0/OSC_IN), Y1.1
- new net BOOT0: IC2.44 (BOOT0), J4.1 (Pin_1), R40.1
- new net USR1: IC2.10 (PA0), TP9.1
- new net USR2: IC2.29 (PA8), TP10.1
- new net VDD_IN_USBCPD: C13.2, IC6.2 (SRC), IC6.3 (IN), IC6.4 (EN), Q1.5 (D), Q3.1 (S), R15.1
Other:
- note added: "(and 6 for C115)"
- note added: "EARTH"
- note added: "Encoder knob - Davies Molding 1101"
- note added: "Version: 0x0000"
- moved on the sheet: C1, C26, C33, C34, C36, C37, C5, C6, D3, H1, H2, J3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

Commit message: update BOM
Parts:
- removed R31: 220, Resistor_SMD:R_0603_1608Metric, symbol Device:R_Small
- added R34: 100, Resistor_SMD:R_0603_1608Metric, symbol Device:R_Small
- C1, C13, C14, C20, C21, C22, C24, C26, C27, C28, C29, C30, C31, C32, C33, C34, C37, C4, C5: Manufacturer_Name Murata Electronics -> KEMET; Manufacturer_Part_Number GRM21BR72A104KAC4L -> C0603C104J5RACTU
- C10, C11: Manufacturer_Name Murata Electronics -> KEMET; Manufacturer_Part_Number GRM2165C1H102JA01D -> C0603C102K3GAC
- C12, C3: Manufacturer_Name Murata Electronics -> KEMET; Manufacturer_Part_Number GRM21A5C2E750FW01D -> C0603C100J5GAC
- C15, C19, C2, C25, C36, C6: Manufacturer_Part_Number GRM21BR6YA106ME43L -> GRM188R6YA106MA73J
- C16, C17, C18: Manufacturer_Name Murata Electronics -> KEMET; Manufacturer_Part_Number GRM21BC72A105KE01L -> C0603C105M8PACTU
- C35, C8, C9: Manufacturer_Name TDK -> Samsung Electro-Mechanics; Manufacturer_Part_Number C2012X6S1C226M125AC -> CL31A226MOCLNNC
- C7: Manufacturer_Name Murata Electronics -> KEMET; Manufacturer_Part_Number GRM21A5C2E750FW01D -> C0603C750K5HACTU
- D5, D6, D7, D8: Mouser Part Number (none) -> 637-BAT54S; Mouser Price/Stock (none) -> https://www.mouser.co.uk/ProductDetail/Diotec-Semiconductor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
- L1: Mouser Part Number e -> 652-SRP7028CC-100M
- Q2: footprint footprints:SOT95P230X110-3N -> SOT95P230X110-3N
- R1, R5: Manufacturer_Part_Number ERJ-6ENF1501V -> ERJ-H3ED1501V; Mouser Part Number (none) -> 667-ERJ-H3ED1501V
- R10: Manufacturer_Part_Number ERJ-6ENF1332V -> ERJ-PB3B1332V; Mouser Part Number (none) -> 667-ERJ-PB3B1332V
- R11, R14: Manufacturer_Part_Number ERJ-6ENF2202V -> ERJ-UP3J223V; Mouser Part Number (none) -> 667-ERJ-UP3J223V
- R12: Manufacturer_Part_Number ERJ-6ENF1003V -> ERJ-P03F1000V; Mouser Part Number (none) -> 667-ERJ-P03F1000V
- R13: Manufacturer_Part_Number ERJ-6ENF2202V -> ERJ-H3EF1001V; Mouser Part Number (none) -> 667-ERJ-H3EF1001V
- R15: Manufacturer_Part_Number ERJ-6ENF1001V -> ERJ-H3EF1001V; Mouser Part Number (none) -> 667-ERJ-H3EF1001V
- R16, R17, R18, R27, R28, R29, R32, R33, R34, R35, R40: Manufacturer_Part_Number ERJ-6ENF1002V -> ERJ-3RBD4701V; Mouser Part Number (none) -> 667-ERJ-3RBD4701V
- R19, R20, R22, R23, R24, R25, R26, R4, R7: Manufacturer_Part_Number ERJ-6ENF4701V -> ERJ-3RBD4701V; Mouser Part Number (none) -> 667-ERJ-3RBD4701V
- R2, R8: Manufacturer_Part_Number ERJ-6ENF4703V -> ERJ-3RED3603V; Mouser Part Number (none) -> 667-ERJ-3RED3603V
- R21: Manufacturer_Part_Number ERJ-6ENF4702V -> ERJ-H3ED4702V; Mouser Part Number (none) -> 667-ERJ-H3ED4702V
- R3, R9: Manufacturer_Part_Number ERJ-6ENF2203V -> ERJ-3RED2203V; Mouser Part Number (none) -> 667-ERJ-3RED2203V
- R30: value 6k8 -> 4k7; Manufacturer_Part_Number ERJ-6ENF6801V -> ERJ-3RBD4701V; Mouser Part Number (none) -> 667-ERJ-3RBD4701V
- R6: Manufacturer_Part_Number ERJ-6ENF1003V -> ERJ-UP3D1003V; Mouser Part Number (none) -> 667-ERJ-UP3D1003V
- U1: Manufacturer_Name (none) -> Adafruit; Manufacturer_Part_Number (none) -> 4311; Mouser Part Number (none) -> 485-4311; Mouser Price/Stock (none) -> https://www.mouser.co.uk/ProductDetail/Adafruit/4311?qs=P1J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
- U4: Mouser Part Number (none) -> 726-BSC014N04LSATMA1
Connections:
- net Buzzer: now also R34.1
- net at Q2.1 (G), R34.1: now also R34.2
Other:
- note added: "24V -> 2.182V"
- note added: "CAPS - AKTSC62K"
- note removed: "24V -> 3,034V"
- moved on the sheet: D12, D3
